File: main_v1.brd (EAGLE design)
At the start: 79.4 x 80.6 mm, 44 parts, among them IC1 MEGA8-P, IC2 LD33V05TV, IC4 MC33063/MC34063P, IC5 MAX6921, IC6 MAX6921

Commit message: Align traces
Routing:
- net GND: track 283.0 -> 281.5 mm
Changed lines of the file:
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@@
 <wire x1="36.5125" y1="26.3525" x2="36.5125" y2="21.9075" width="0.4064" layer="1"/>
 <via x="36.5125" y="21.9075" extent="1-16" drill="0.8128" diameter="1.27" shape="octagon"/>
-<via x="33.9725" y="49.8475" extent="1-16" drill="0.8128" diameter="1.27" shape="octagon"/>
-<via x="21.2725" y="49.8475" extent="1-16" drill="0.8128" diameter="1.27" shape="octagon"/>
-<wire x1="21.2725" y1="49.8475" x2="33.9725" y2="49.8475" width="0.4064" layer="1"/>
+<via x="33.655" y="50.4825" extent="1-16" drill="0.8128" diameter="1.27" shape="octagon"/>
+<via x="21.2725" y="50.4825" extent="1-16" drill="0.8128" diameter="1.27" shape="octagon"/>
+<wire x1="21.2725" y1="50.4825" x2="33.655" y2="50.4825" width="0.4064" layer="1"/>
 <contactref element="IC3" pad="1"/>
 <contactref element="IC3" pad="3"/>
@@
 <wire x1="37.7825" y1="72.0725" x2="37.7825" y2="69.5325" width="0.4064" layer="16"/>
 <wire x1="37.7825" y1="69.5325" x2="36.83" y2="68.58" width="0.4064" layer="16"/>
-<wire x1="21.2725" y1="49.8475" x2="21.2725" y2="50.8" width="1.016" layer="16"/>
+<wire x1="21.2725" y1="50.4825" x2="21.2725" y2="50.8" width="1.016" layer="16"/>
 <wire x1="34.925" y1="45.72" x2="33.655" y2="46.99" width="0.4064" layer="16"/>
 <wire x1="33.655" y1="46.99" x2="33.02" y2="46.99" width="0.4064" layer="16"/>
 <wire x1="33.02" y1="46.99" x2="32.385" y2="47.625" width="0.4064" layer="16"/>
 <wire x1="32.385" y1="47.625" x2="32.385" y2="49.53" width="0.4064" layer="16"/>
-<wire x1="32.385" y1="49.53" x2="32.7025" y2="49.8475" width="0.4064" layer="16"/>
-<wire x1="32.7025" y1="49.8475" x2="33.9725" y2="49.8475" width="0.4064" layer="16"/>
-<wire x1="33.9725" y1="49.8475" x2="34.29" y2="50.165" width="0.4064" layer="16"/>
+<wire x1="32.385" y1="49.53" x2="33.3375" y2="50.4825" width="0.4064" layer="16"/>
+<wire x1="33.3375" y1="50.4825" x2="33.655" y2="50.4825" width="0.4064" layer="16"/>
+<wire x1="33.655" y1="50.4825" x2="34.29" y2="51.1175" width="0.4064" layer="16"/>
 <wire x1="31.75" y1="58.42" x2="31.75" y2="55.245" width="0.4064" layer="16"/>
 <wire x1="31.75" y1="55.245" x2="32.385" y2="54.61" width="0.4064" layer="16"/>
 <wire x1="32.385" y1="54.61" x2="33.655" y2="54.61" width="0.4064" layer="16"/>
 <wire x1="33.655" y1="54.61" x2="34.29" y2="53.975" width="0.4064" layer="16"/>
-<wire x1="34.29" y1="53.975" x2="34.29" y2="50.165" width="0.4064" layer="16"/>
+<wire x1="34.29" y1="53.975" x2="34.29" y2="51.1175" width="0.4064" layer="16"/>
 <wire x1="39.37" y1="63.5" x2="36.83" y2="66.04" width="0.4064" layer="16"/>
 <wire x1="36.83" y1="66.04" x2="36.83" y2="68.58" width="0.4064" layer="16"/>
