File: main_v2.sch (EAGLE design)
At the start: 28 parts, among them IC1 MAX6921, IC2 MAX6921, IC3 MC33063, IC4 LD33V05T, IC5 TDA7052A

Commit message: More work on the board
Connections:
- net GATE4: now also IC1.OUT1; no longer IC1.OUT9
- net OUT24: now also IC1.OUT3; no longer IC1.OUT0
- net OUT25: now also IC1.OUT5; no longer IC1.OUT1
- net OUT26: now also IC1.OUT4; no longer IC1.OUT2
- net OUT27: now also IC1.OUT7; no longer IC1.OUT3
- net OUT28: now also IC1.OUT6; no longer IC1.OUT4
- net OUT29: now also IC1.OUT8; no longer IC1.OUT5
- net OUT30: now also IC1.OUT9; no longer IC1.OUT6
- net OUT31: now also IC1.OUT2; no longer IC1.OUT7
- net SPARE4: now also IC1.OUT0; no longer IC1.OUT8
Changed lines of the file:
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@@
 </segment>
 <segment>
-<pinref part="IC1" gate="G$1" pin="OUT0"/>
-<wire x1="147.32" y1="160.02" x2="157.48" y2="160.02" width="0.1524" layer="91"/>
+<pinref part="IC1" gate="G$1" pin="OUT3"/>
+<wire x1="157.48" y1="152.4" x2="147.32" y2="152.4" width="0.1524" layer="91"/>
 </segment>
 </net>
@@
 </segment>
 <segment>
-<pinref part="IC1" gate="G$1" pin="OUT2"/>
-<wire x1="147.32" y1="154.94" x2="157.48" y2="154.94" width="0.1524" layer="91"/>
+<pinref part="IC1" gate="G$1" pin="OUT4"/>
+<wire x1="157.48" y1="149.86" x2="147.32" y2="149.86" width="0.1524" layer="91"/>
 </segment>
 </net>
@@
 </segment>
 <segment>
-<pinref part="IC1" gate="G$1" pin="OUT3"/>
-<wire x1="147.32" y1="152.4" x2="157.48" y2="152.4" width="0.1524" layer="91"/>
+<pinref part="IC1" gate="G$1" pin="OUT7"/>
+<wire x1="157.48" y1="142.24" x2="147.32" y2="142.24" width="0.1524" layer="91"/>
 </segment>
 </net>
@@
 </segment>
 <segment>
-<pinref part="IC1" gate="G$1" pin="OUT4"/>
-<wire x1="147.32" y1="149.86" x2="157.48" y2="149.86" width="0.1524" layer="91"/>
+<pinref part="IC1" gate="G$1" pin="OUT6"/>
+<wire x1="157.48" y1="144.78" x2="147.32" y2="144.78" width="0.1524" layer="91"/>
 </segment>
 </net>
@@
 </segment>
 <segment>
-<pinref part="IC1" gate="G$1" pin="OUT5"/>
-<wire x1="147.32" y1="147.32" x2="157.48" y2="147.32" width="0.1524" layer="91"/>
+<pinref part="IC1" gate="G$1" pin="OUT8"/>
+<wire x1="157.48" y1="139.7" x2="147.32" y2="139.7" width="0.1524" layer="91"/>
 </segment>
 </net>
@@
 </segment>
 <segment>
-<pinref part="IC1" gate="G$1" pin="OUT6"/>
-<wire x1="147.32" y1="144.78" x2="157.48" y2="144.78" width="0.1524" layer="91"/>
+<pinref part="IC1" gate="G$1" pin="OUT9"/>
+<wire x1="157.48" y1="137.16" x2="147.32" y2="137.16" width="0.1524" layer="91"/>
 </segment>
 </net>
@@
 </segment>
 <segment>
-<pinref part="IC1" gate="G$1" pin="OUT7"/>
-<wire x1="147.32" y1="142.24" x2="157.48" y2="142.24" width="0.1524" layer="91"/>
+<pinref part="IC1" gate="G$1" pin="OUT2"/>
+<wire x1="157.48" y1="154.94" x2="147.32" y2="154.94" width="0.1524" layer="91"/>
 </segment>
 </net>
@@
 </segment>
 <segment>
-<pinref part="IC1" gate="G$1" pin="OUT1"/>
-<wire x1="147.32" y1="157.48" x2="157.48" y2="157.48" width="0.1524" layer="91"/>
+<pinref part="IC1" gate="G$1" pin="OUT5"/>
+<wire x1="157.48" y1="147.32" x2="147.32" y2="147.32" width="0.1524" layer="91"/>
 </segment>
 </net>
@@
 </segment>
 <segment>
-<pinref part="IC1" gate="G$1" pin="OUT9"/>
-<wire x1="147.32" y1="137.16" x2="157.48" y2="137.16" width="0.1524" layer="91"/>
+<pinref part="IC1" gate="G$1" pin="OUT1"/>
+<wire x1="157.48" y1="157.48" x2="147.32" y2="157.48" width="0.1524" layer="91"/>
 </segment>
 </net>
@@
 </segment>
 <segment>
-<pinref part="IC1" gate="G$1" pin="OUT8"/>
-<wire x1="147.32" y1="139.7" x2="157.48" y2="139.7" width="0.1524" layer="91"/>
-</segment>
-</net>
+<pinref part="IC1" gate="G$1" pin="OUT0"/>
+<wire x1="157.48" y1="160.02" x2="147.32" y2="160.02" width="0.1524" layer="91"/>
+</segment>
+</net>

Commit message: Nearly there
Connections:
- net N$3: now also SPI.2; no longer SPI.4
- net SCK: now also SPI.4; no longer SPI.2
Changed lines of the file:
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@@
 <wire x1="71.12" y1="144.78" x2="104.14" y2="144.78" width="0.1524" layer="91"/>
 <junction x="104.14" y="144.78"/>
-<pinref part="SPI" gate="G$1" pin="2"/>
-<wire x1="86.36" y1="167.64" x2="71.12" y2="167.64" width="0.1524" layer="91"/>
-<wire x1="71.12" y1="167.64" x2="71.12" y2="144.78" width="0.1524" layer="91"/>
+<wire x1="71.12" y1="144.78" x2="71.12" y2="162.56" width="0.1524" layer="91"/>
+<pinref part="SPI" gate="G$1" pin="4"/>
+<wire x1="71.12" y1="162.56" x2="86.36" y2="162.56" width="0.1524" layer="91"/>
 </segment>
 </net>
@@
 <wire x1="109.22" y1="134.62" x2="66.04" y2="134.62" width="0.1524" layer="91"/>
 <junction x="109.22" y="134.62"/>
-<wire x1="66.04" y1="134.62" x2="66.04" y2="162.56" width="0.1524" layer="91"/>
-<pinref part="SPI" gate="G$1" pin="4"/>
-<wire x1="66.04" y1="162.56" x2="86.36" y2="162.56" width="0.1524" layer="91"/>
+<wire x1="66.04" y1="134.62" x2="66.04" y2="167.64" width="0.1524" layer="91"/>
+<pinref part="SPI" gate="G$1" pin="2"/>
+<wire x1="66.04" y1="167.64" x2="86.36" y2="167.64" width="0.1524" layer="91"/>
 </segment>
 </net>
@@
 <wire x1="106.68" y1="139.7" x2="68.58" y2="139.7" width="0.1524" layer="91"/>
 <junction x="106.68" y="139.7"/>
-<wire x1="68.58" y1="139.7" x2="68.58" y2="165.1" width="0.1524" layer="91"/>
 <pinref part="SPI" gate="G$1" pin="3"/>
-<wire x1="68.58" y1="165.1" x2="86.36" y2="165.1" width="0.1524" layer="91"/>
+<wire x1="86.36" y1="165.1" x2="68.58" y2="165.1" width="0.1524" layer="91"/>
+<wire x1="68.58" y1="165.1" x2="68.58" y2="139.7" width="0.1524" layer="91"/>
 </segment>
 </net>

Commit message: Try SPI header vertically
Connections:
- net MOSI: now also SPI.4; no longer SPI.1
- net N$3: now also SPI.1; no longer SPI.2
- net SCK: now also SPI.2; no longer SPI.4
Changed lines of the file:
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@@
 <pinref part="IC1" gate="G$1" pin="DIN"/>
 <wire x1="114.3" y1="149.86" x2="73.66" y2="149.86" width="0.1524" layer="91"/>
-<wire x1="73.66" y1="149.86" x2="73.66" y2="170.18" width="0.1524" layer="91"/>
-<pinref part="SPI" gate="G$1" pin="1"/>
-<wire x1="73.66" y1="170.18" x2="86.36" y2="170.18" width="0.1524" layer="91"/>
+<wire x1="73.66" y1="149.86" x2="73.66" y2="162.56" width="0.1524" layer="91"/>
+<pinref part="SPI" gate="G$1" pin="4"/>
+<wire x1="73.66" y1="162.56" x2="86.36" y2="162.56" width="0.1524" layer="91"/>
 </segment>
 </net>
@@
 <wire x1="71.12" y1="144.78" x2="104.14" y2="144.78" width="0.1524" layer="91"/>
 <junction x="104.14" y="144.78"/>
-<wire x1="71.12" y1="144.78" x2="71.12" y2="162.56" width="0.1524" layer="91"/>
-<pinref part="SPI" gate="G$1" pin="4"/>
-<wire x1="71.12" y1="162.56" x2="86.36" y2="162.56" width="0.1524" layer="91"/>
+<wire x1="71.12" y1="144.78" x2="71.12" y2="167.64" width="0.1524" layer="91"/>
+<pinref part="SPI" gate="G$1" pin="2"/>
+<wire x1="71.12" y1="167.64" x2="86.36" y2="167.64" width="0.1524" layer="91"/>
 </segment>
 </net>
@@
 <wire x1="109.22" y1="134.62" x2="66.04" y2="134.62" width="0.1524" layer="91"/>
 <junction x="109.22" y="134.62"/>
-<wire x1="66.04" y1="134.62" x2="66.04" y2="167.64" width="0.1524" layer="91"/>
-<pinref part="SPI" gate="G$1" pin="2"/>
-<wire x1="66.04" y1="167.64" x2="86.36" y2="167.64" width="0.1524" layer="91"/>
+<wire x1="66.04" y1="134.62" x2="66.04" y2="170.18" width="0.1524" layer="91"/>
+<pinref part="SPI" gate="G$1" pin="1"/>
+<wire x1="66.04" y1="170.18" x2="86.36" y2="170.18" width="0.1524" layer="91"/>
 </segment>
 </net>
@@
 <wire x1="106.68" y1="139.7" x2="68.58" y2="139.7" width="0.1524" layer="91"/>
 <junction x="106.68" y="139.7"/>
+<wire x1="68.58" y1="165.1" x2="68.58" y2="139.7" width="0.1524" layer="91"/>
 <pinref part="SPI" gate="G$1" pin="3"/>
-<wire x1="86.36" y1="165.1" x2="68.58" y2="165.1" width="0.1524" layer="91"/>
-<wire x1="68.58" y1="165.1" x2="68.58" y2="139.7" width="0.1524" layer="91"/>
+<wire x1="68.58" y1="165.1" x2="86.36" y2="165.1" width="0.1524" layer="91"/>
 </segment>
 </net>

Commit message: Well, its finished
Connections:
- net MOSI: now also SPI.1; no longer SPI.4
- net N$3: now also SPI.2; no longer SPI.1
- net SCK: now also SPI.4; no longer SPI.2
Changed lines of the file:
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@@
 </instances>
 <busses>
-<bus name="OUT[0..32],HT+[1..4],HT-[1..4],GATE[1..4],SPARE[1..4]">
+<bus name="OUT[0..32],HT+[1..4],HT-,HT+,GATE[1..4],SPARE[1..4]">
 <segment>
 <wire x1="157.48" y1="15.24" x2="193.04" y2="15.24" width="0.762" layer="92"/>
@@
 <pinref part="IC1" gate="G$1" pin="DIN"/>
 <wire x1="114.3" y1="149.86" x2="73.66" y2="149.86" width="0.1524" layer="91"/>
-<wire x1="73.66" y1="149.86" x2="73.66" y2="162.56" width="0.1524" layer="91"/>
-<pinref part="SPI" gate="G$1" pin="4"/>
-<wire x1="73.66" y1="162.56" x2="86.36" y2="162.56" width="0.1524" layer="91"/>
+<wire x1="73.66" y1="149.86" x2="73.66" y2="170.18" width="0.1524" layer="91"/>
+<pinref part="SPI" gate="G$1" pin="1"/>
+<wire x1="73.66" y1="170.18" x2="86.36" y2="170.18" width="0.1524" layer="91"/>
 </segment>
 </net>
@@
 <wire x1="71.12" y1="144.78" x2="104.14" y2="144.78" width="0.1524" layer="91"/>
 <junction x="104.14" y="144.78"/>
-<wire x1="71.12" y1="144.78" x2="71.12" y2="167.64" width="0.1524" layer="91"/>
-<pinref part="SPI" gate="G$1" pin="2"/>
-<wire x1="71.12" y1="167.64" x2="86.36" y2="167.64" width="0.1524" layer="91"/>
+<wire x1="71.12" y1="144.78" x2="71.12" y2="162.56" width="0.1524" layer="91"/>
+<pinref part="SPI" gate="G$1" pin="4"/>
+<wire x1="71.12" y1="162.56" x2="86.36" y2="162.56" width="0.1524" layer="91"/>
 </segment>
 </net>
@@
 <wire x1="109.22" y1="134.62" x2="66.04" y2="134.62" width="0.1524" layer="91"/>
 <junction x="109.22" y="134.62"/>
-<wire x1="66.04" y1="134.62" x2="66.04" y2="170.18" width="0.1524" layer="91"/>
-<pinref part="SPI" gate="G$1" pin="1"/>
-<wire x1="66.04" y1="170.18" x2="86.36" y2="170.18" width="0.1524" layer="91"/>
+<wire x1="66.04" y1="134.62" x2="66.04" y2="167.64" width="0.1524" layer="91"/>
+<pinref part="SPI" gate="G$1" pin="2"/>
+<wire x1="66.04" y1="167.64" x2="86.36" y2="167.64" width="0.1524" layer="91"/>
 </segment>
 </net>
@@
 <wire x1="106.68" y1="139.7" x2="68.58" y2="139.7" width="0.1524" layer="91"/>
 <junction x="106.68" y="139.7"/>
+<pinref part="SPI" gate="G$1" pin="3"/>
+<wire x1="86.36" y1="165.1" x2="68.58" y2="165.1" width="0.1524" layer="91"/>
 <wire x1="68.58" y1="165.1" x2="68.58" y2="139.7" width="0.1524" layer="91"/>
-<pinref part="SPI" gate="G$1" pin="3"/>
-<wire x1="68.58" y1="165.1" x2="86.36" y2="165.1" width="0.1524" layer="91"/>
-</segment>
-</net>
+</segment>
+</net>
