File: main_v2.brd (EAGLE design)
At the start: 76.8 x 39.4 mm, 28 parts, among them IC1 MAX6921, IC2 MAX6921, IC3 MC33063, IC4 LD33V05T, IC5 TDA7052A

Commit message: Final Touches
Parts:
- moved C5 18.4 mm to (72.1, 11.1), turned to 90 degrees
- moved C4 16.7 mm to (70.2, 28.3)
- moved R1 0.90 mm to (69.5, 9.21)
- moved R5 0.64 mm to (19.7, 32.4)
- moved C2 0.64 mm to (28.6, 28.6)
- moved C3 0.64 mm to (25.4, 17.1)
- moved C6 0.64 mm to (10.8, 22.9)
- moved C7 0.64 mm to (5.08, 21.6)
- moved C8 0.64 mm to (21.0, 17.1)
- moved D3 0.64 mm to (6.99, 27.3)
- moved H3 0.64 mm to (56.5, 24.1)
- moved IC1 0.64 mm to (39.4, 28.6)
- moved IC3 0.64 mm to (18.4, 25.4)
- moved R6 0.64 mm to (25.1, 26.0)
- moved R7 0.64 mm to (13.3, 15.9)
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Routing:
- net VCC: track 152.3 -> 135.9 mm
- net N$12: track 4.97 -> 14.2 mm
- net GND: track 203.6 -> 211.8 mm
- net N$10: track 7.88 -> 13.8 mm
- net N$3: track 81.1 -> 79.1 mm
- net N$4: track 76.2 -> 75.0 mm
Other:
- board size 76.8 x 39.4 mm -> 76.8 x 38.7 mm
- board text added: "KJ-22 Apr 2021"
- board text added: "YT"
- board text removed: "YT KJ-22 Apr 2021"
